File: kicad_proj/test_kibot.kicad_pcb (KiCad board)
At the start: 4 copper layers, 51.7 x 41 mm, 41 parts, among them J1 _GENERIC_CONNECTOR_01x02, J2 1988804, Q1 TPH3R704PL,L1Q, Q2 TPH3R704PL,L1Q, Q3 TPH3R704PL,L1Q, Q4 TPH3R704PL,L1Q, U1 MC78M12BDTG, U2 74HCT2G14GV,125, U3 MC78M05CDTRKG, U4 DGD0506AM10-13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

Commit message: New outline
Parts:
- removed C1, C10, C11, C12, C13, C3, C4, C5: GRM188R61H225ME11D, footprints:CAPACITOR_0603N
- removed C14, C15: GRM32EC72A106KE05L, footprints:CAPACITOR_1210N
- removed C2: CL10B103KB8NNNC, footprints:CAPACITOR_0603N
- removed C6, C7: CL10A475KA8NQNC, footprints:CAPACITOR_0603N
- removed C8, C9: CC0603KRX7R9BB104, footprints:CAPACITOR_0603N
- removed J2: 1988804, footprints:1988804
- removed Q1, Q2, Q3, Q4: TPH3R704PL,L1Q, footprints:2-5Q1S
- removed R1: RC0603JR-07470RL, footprints:RESISTOR_0603N
- removed R10, R7, R8, R9: RC0603JR-0720RL, footprints:RESISTOR_0603N
- removed R2: RC0603FR-07174RL, footprints:RESISTOR_0603N
- removed R3, R4: RC0603JR-070RL, footprints:RESISTOR_0603N
- removed R5, R6: RC0603JR-07100KL, footprints:RESISTOR_0603N
- removed REF** (x5): MountingHole_3.2mm_M3, MountingHole:MountingHole_3.2mm_M3
- removed U1: MC78M12BDTG, footprints:DPAK4P229_990X238L159X76T520X546N
- removed U2: 74HCT2G14GV,125, footprints:SOP6P95_290X275X110L40X32N
- removed U3: MC78M05CDTRKG, footprints:DPAK4P229_990X238L159X76T520X546N
- removed U4, U5: DGD0506AM10-13, footprints:SOP10P50_300X490X110L60X22N
- added H1: MountingHole_Pad, footprints:MountingHole_3.2mm_M3_Pad_Via, F.Cu at (130.6, 34.7)
- added H2: MountingHole_Pad, footprints:MountingHole_3.2mm_M3_Pad_Via, F.Cu at (122.9, 34.7)
- added H3: MountingHole_Pad, footprints:MountingHole_3.2mm_M3_Pad_Via, F.Cu at (162.3, 34.7)
- added H4: MountingHole_Pad, footprints:MountingHole_3.2mm_M3_Pad_Via, F.Cu at (170.0, 34.7)
- added TP2: TestPoint, TestPoint:TestPoint_Pad_2.0x2.0mm, F.Cu at (166.2, 38.8)
- J1: value _GENERIC_CONNECTOR_01x02 -> 5023520300; footprint footprints:B2B-XH-A(LF)(SN) -> footprints:5023520300
- moved J1 3.90 mm to (126.3, 44.1), turned to 0 degrees
Connections:
- J1 pad 1: +24V -> (no net)
- J1 pad 2: GND -> (no net)
Routing:
- net +12V: track 84.3 -> 10.2 mm, vias 2 -> 0
- net +24V: track 65.3 -> 0.00 mm, vias 16 -> 0
- net +5V: track 82.9 -> 18.4 mm, vias 8 -> 1
- net GND: track 58.2 -> 0.88 mm, vias 69 -> 9
- net Net-(U4-Pad8): track 37.4 -> 5.80 mm, vias 2 -> 0
- net Net-(C9-Pad2): track 30.3 -> 0.00 mm
- net /DRIVE: track 31.4 -> 1.93 mm, vias 2 -> 0
- net Net-(C8-Pad2): track 17.2 -> 0.00 mm
- net Net-(R7-Pad1): track 7.11 -> 0.00 mm
- net Net-(R6-Pad1): track 6.93 -> 0.00 mm
- net Net-(R10-Pad1): track 5.14 -> 0.00 mm
- net Net-(R8-Pad1): track 5.04 -> 0.00 mm
- net Net-(C9-Pad1): track 4.65 -> 0.00 mm
- net Net-(R9-Pad1): track 4.39 -> 0.00 mm
- net Net-(C8-Pad1): track 3.85 -> 0.00 mm
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- added copper zone on B.Cu, net (none)
Other:
- board size 51.7 x 41 mm -> 54 x 22.2 mm
- board text removed: "24V"
- board text removed: "GND"
- board text removed: "MULTIPLE UNIT MIST V1a"

Commit message: Changes pours
Routing:
- net +5V: track 18.4 -> 5.51 mm
- net +12V: track 10.2 -> 0.00 mm
- net Net-(U4-Pad8): track 5.80 -> 0.00 mm
- net /DRIVE: track 1.93 -> 0.00 mm
- removed copper zone on B.Cu, net (none)
- removed copper zone on B.Cu, net +24V
Changed lines of the file:
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@@
   (net 1 "GND")
   (net 2 "+5V")
-  (net 3 "+24V")
-  (net 4 "+12V")
-  (net 5 "/DRIVE")
-  (net 6 "Net-(U4-Pad8)")
   (footprint "TestPoint:TestPoint_Pad_2.0x2.0mm" (layer "F.Cu")
     (at 166.2 38.8)
@@
   (segment (start 133.1 51.4) (end 133.36 51.14) (width 0.4) (layer "F.Cu") (net 2))
   (via (at 133.1 51.4) (size 0.8) (drill 0.4) (layers "F.Cu" "B.Cu") (net 2))
-  (segment (start 170.920355 28) (end 169 28) (width 0.3) (layer "B.Cu") (net 2))
-  (segment (start 169 28) (end 168.8 28.2) (width 0.3) (layer "B.Cu") (net 2))
   (segment (start 141.5 39.8) (end 141.5 37.7) (width 0.3) (layer "B.Cu") (net 2))
-  (segment (start 158.92172 60.0893) (end 156.2107 60.0893) (width 0.3) (layer "B.Cu") (net 2))
-  (segment (start 168.8 28.2) (end 168.5 28.5) (width 0.3) (layer "B.Cu") (net 2))
-  (segment (start 168.5 28.5) (end 161 28.5) (width 0.3) (layer "B.Cu") (net 2))
-  (segment (start 156.2107 60.0893) (end 156.2 60.1) (width 0.3) (layer "B.Cu") (net 2))
   (segment (start 148.5 40.4) (end 146.2 40.4) (width 0.3) (layer "B.Cu") (net 2))
-  (segment (start 163.7 63.4) (end 159.3 63.4) (width 0.5) (layer "B.Cu") (net 4))
-  (segment (start 159.3 63.4) (end 153.5 63.4) (width 0.5) (layer "B.Cu") (net 4))
-  (segment (start 157.208969 61.308969) (end 158.985643 61.308969) (width 0.25) (layer "B.Cu") (net 5))
-  (segment (start 157.1 61.2) (end 157.208969 61.308969) (width 0.25) (layer "B.Cu") (net 5))
-  (segment (start 167.5 27.5) (end 161.7 27.5) (width 0.25) (layer "B.Cu") (net 6))
   (zone (net 1) (net_name "GND") (layers "F.Cu" "In1.Cu" "In2.Cu") (hatch edge 0.508)
     (connect_pads (clearance 0.2))
@@
       )
     )
-  )
-  (zone (net 0) (net_name "") (layer "B.Cu") (hatch edge 0.508)
-    (connect_pads (clearance 0.2))
-    (min_thickness 0.2) (filled_areas_thickness no)
-    (fill yes (thermal_gap 0.508) (thermal_bridge_width 0.508))
-    (polygon
-      (pts
-        (xy 177.3 91.5)
-        (xy 123.5 91.5)
-        (xy 123.5 69.5)
-        (xy 177.3 69.5)
-      )
-    )
-  )
-  (zone (net 3) (net_name "+24V") (layer "B.Cu") (hatch edge 0.508)
-    (connect_pads (clearance 0.2))
-    (min_thickness 0.2) (filled_areas_thickness no)
-    (fill yes (thermal_gap 0.2) (thermal_bridge_width 0.25))
-    (polygon
-      (pts
-        (xy 176.5 65)
-        (xy 124.8 65)
-        (xy 124.8 24)
-        (xy 176.49339 24)
-      )
-    )
